File: circuits/lighthouse/lighthouse.kicad_sch (KiCad schematic)
At the start: 56 parts, among them J1 USB_C_Receptacle_USB2.0_14P, J2 Conn_01x03_Socket, Q1 S9013, Q4 SS8050, Q5 SS8050, U10 CP2102-GMR, U2 AMS1117-3.3, U7 ESP32-WROOM-32

Commit message: Safekeeping
Parts:
- removed S1: SLW-1678105-6A-N-D, SLW-1678105-6A-N-D:SLW16781056AND, symbol SLW-1678105-6A-N-D:SLW-1678105-6A-N-D
- added SW1: SW_Push_DPDT, Connector_JST:JST_XH_B4B-XH-A_1x04_P2.50mm_Vertical, symbol Switch:SW_Push_DPDT
- D1, D2, D3, D4: footprint LED_SMD:LED_1206_3216Metric_Pad1.42x1.75mm_HandSolder -> LED_THT:LED_D3.0mm
- Q1: value S9013 -> BC337
- Q4, Q5: value SS8050 -> BC817-40
- R4: value 240 -> 150
- R7: value 10k -> 100k
- R9: value 20k -> 47k
Connections:
- net Charger/+OUT: now also SW1.1 (B)
- net Charger/VIN: now also SW1.4 (B)
- net at F2.1: now also SW1.2 (A)
- net at F1.1: now also SW1.3
Changed lines of the file:
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@@
 	)
 	(junction
-		(at 120.65 90.17)
-		(diameter 0)
-		(color 0 0 0 0)
-	)
-	(junction
 		(at 259.08 92.71)
 		(diameter 0)
@@
 	(wire
 		(pts
+			(xy 210.82 34.29) (xy 210.82 36.83)
+		)
+		(stroke
+			(width 0)
+			(type default)
+		)
+	)
+	(wire
+		(pts
 			(xy 76.2 168.91) (xy 76.2 176.53)
 		)
@@
 	(wire
 		(pts
-			(xy 173.99 36.83) (xy 185.42 36.83)
+			(xy 173.99 36.83) (xy 193.04 36.83)
 		)
 		(stroke
@@
 	(wire
 		(pts
-			(xy 120.65 90.17) (xy 123.19 90.17)
+			(xy 184.15 72.39) (xy 187.96 72.39)
 		)
 		(stroke
@@
 	(wire
 		(pts
-			(xy 184.15 72.39) (xy 187.96 72.39)
+			(xy 210.82 24.13) (xy 210.82 26.67)
 		)
 		(stroke
@@
 	(wire
 		(pts
-			(xy 119.38 90.17) (xy 120.65 90.17)
-		)
-		(stroke
-			(width 0)
-			(type default)
-		)
-	)
-	(wire
-		(pts
 			(xy 60.96 35.56) (xy 77.47 35.56)
 		)
@@
 	(wire
 		(pts
+			(xy 120.65 90.17) (xy 123.19 90.17)
+		)
+		(stroke
+			(width 0)
+			(type default)
+		)
+	)
+	(wire
+		(pts
 			(xy 60.96 27.94) (xy 66.04 27.94)
 		)
@@
 	(wire
 		(pts
+			(xy 203.2 24.13) (xy 210.82 24.13)
+		)
+		(stroke
+			(width 0)
+			(type default)
+		)
+	)
+	(wire
+		(pts
 			(xy 49.53 109.22) (xy 49.53 104.14)
 		)
@@
 	(wire
 		(pts
+			(xy 203.2 34.29) (xy 210.82 34.29)
+		)
+		(stroke
+			(width 0)
+			(type default)
+		)
+	)
+	(wire
+		(pts
 			(xy 49.53 104.14) (xy 50.8 104.14)
 		)
@@
 	(wire
 		(pts
-			(xy 142.24 26.67) (xy 185.42 26.67)
+			(xy 142.24 26.67) (xy 193.04 26.67)
 		)
 		(stroke
@@
 			)
 		)
-		(property "Footprint" "LED_SMD:LED_1206_3216Metric_Pad1.42x1.75mm_HandSolder"
+		(property "Footprint" "LED_THT:LED_D3.0mm"
 			(at 52.07 161.29 0)
 			(effects
@@
 			)
 		)
-		(property "Value" "S9013"
+		(property "Value" "BC337"
 			(at 139.7 173.9899 0)
 			(effects
@@
 			)
 		)
-		(property "Value" "240"
+		(property "Value" "150"
 			(at 121.92 168.91 90)
 			(effects
@@
 			)
 		)
-		(property "Footprint" "LED_SMD:LED_1206_3216Metric_Pad1.42x1.75mm_HandSolder"
+		(property "Footprint" "LED_THT:LED_D3.0mm"
 			(at 52.07 184.15 0)
 			(effects
@@
 			)
 		)
-		(property "Value" "SS8050"
+		(property "Value" "BC817-40"
 			(at 71.12 105.4099 0)
 			(effects
@@
 			)
 		)
-		(property "Value" "10k"
+		(property "Value" "100k"
 			(at 121.92 154.9401 0)
 			(effects
@@
 			)
 		)
-		(property "Value" "SS8050"
+		(property "Value" "BC817-40"
 			(at 46.99 115.5699 0)
 			(effects
@@
 			)
 		)
-		(property "Footprint" "LED_SMD:LED_1206_3216Metric_Pad1.42x1.75mm_HandSolder"
+		(property "Footprint" "LED_THT:LED_D3.0mm"
 			(at 52.07 176.53 0)
 			(effects
@@
 			)
 		)
-		(property "Value" "20k"
+		(property "Value" "47k"
 			(at 121.92 142.2401 0)
 			(effects
@@
 	)
 	(symbol
-		(lib_id "Device:R")
-		(at 67.31 184.15 90)
+		(lib_id "Switch:SW_Push_DPDT")
+		(at 198.12 31.75 0)
 		(unit 1)
 		(exclude_from_sim no)
@@
 		(on_board yes)
 		(dnp no)
-		(property "Reference" "R13"
-			(at 67.31 181.61 90)
+		(fields_autoplaced yes)
+		(property "Reference" "SW1"
+			(at 198.12 17.78 0)
 			(effects
 				(font
@@
 			)
 		)
-		(property "Value" "1k"
-			(at 67.564 186.944 90)
+		(property "Value" "SW_Push_DPDT"
+			(at 198.12 20.32 0)
 			(effects
 				(font
@@
 			)
 		)
-		(property "Footprint" "Resistor_SMD:R_1206_3216Metric_Pad1.30x1.75mm_HandSolder"
-			(at 67.31 185.928 90)
+		(property "Footprint" "Connector_JST:JST_XH_B4B-XH-A_1x04_P2.50mm_Vertical"
+			(at 198.12 26.67 0)
 			(effects
 				(font
@@
 		)
 		(property "Datasheet" "~"
-			(at 67.31 184.15 0)
+			(at 198.12 26.67 0)
 			(effects
 				(font
@@
 			)
 		)
-		(property "Description" "Resistor"
-			(at 67.31 184.15 0)
+		(property "Description" "Momentary Switch, dual pole double throw"
+			(at 198.12 31.75 0)
 			(effects
 				(font
@@
 		(pin "1"
 		)
+		(pin "5"
+		)
+		(pin "4"
+		)
 		(pin "2"
 		)
+		(pin "3"
+		)
+		(pin "6"
+		)
 		(instances
 			(project ""
 				(path "/7210d03b-7565-45ff-aaca-ad566f37cd67"
-					(reference "R13")
+					(reference "SW1")
 					(unit 1)
 				)
@@
 	(symbol
 		(lib_id "Device:R")
-		(at 88.9 66.04 90)
+		(at 67.31 184.15 90)
 		(unit 1)
 		(exclude_from_sim no)
@@
 		(on_board yes)
 		(dnp no)
-		(property "Reference" "R34"
-			(at 87.0153 71.2429 90)
+		(property "Reference" "R13"
+			(at 67.31 181.61 90)
 			(effects
 				(font
 					(size 1.27 1.27)
 				)
-				(justify right)
 			)
 		)
-		(property "Value" "10k"
-			(at 87.0153 68.7029 90)
+		(property "Value" "1k"
+			(at 67.564 186.944 90)
 			(effects
 				(font
 					(size 1.27 1.27)
 				)
-				(justify right)
 			)
 		)
 		(property "Footprint" "Resistor_SMD:R_1206_3216Metric_Pad1.30x1.75mm_HandSolder"
-			(at 88.9 67.818 90)
+			(at 67.31 185.928 90)
 			(effects
 				(font
@@
 		)
 		(property "Datasheet" "~"
-			(at 88.9 66.04 0)
+			(at 67.31 184.15 0)
 			(effects
 				(font
@@
 		)
 		(property "Description" "Resistor"
-			(at 88.9 66.04 0)
+			(at 67.31 184.15 0)
 			(effects
 				(font
@@
 		)
 		(instances
-			(project "lighthouse"
+			(project ""
 				(path "/7210d03b-7565-45ff-aaca-ad566f37cd67"
-					(reference "R34")
+					(reference "R13")
 					(unit 1)
 				)
@@
 	)
 	(symbol
-		(lib_id "SLW-1678105-6A-N-D:SLW-1678105-6A-N-D")
-		(at 185.42 26.67 0)
+		(lib_id "Device:R")
+		(at 88.9 66.04 90)
 		(unit 1)
 		(exclude_from_sim no)
@@
 		(on_board yes)
 		(dnp no)
-		(property "Reference" "S1"
-			(at 198.12 19.05 0)
-			(effects
-				(font
-					(size 1.27 1.27)
-				)
-			)
-		)
-		(property "Value" "SLW-1678105-6A-N-D"
-			(at 198.12 21.59 0)
-			(effects
-				(font
-					(size 1.27 1.27)
-				)
-			)
-		)
-		(property "Footprint" "SLW-1678105-6A-N-D:SLW16781056AND"
-			(at 184.15 121.59 0)
-			(effects
-				(font
-					(size 1.27 1.27)
-				)
-				(justify left top)
-				(hide yes)
-			)
-		)
-		(property "Datasheet" "https://www.sameskydevices.com/product/resource/SLW-1678105-6A-N-D.pdf"
-			(at 184.15 221.59 0)
-			(effects
-				(font
-					(size 1.27 1.27)
-				)
-				(justify left top)
-				(hide yes)
-			)
-		)
-		(property "Description" "SLW-1678105-6A-N-D - 16 x 7.8 x 10.5 mm, 6 mm Raised Slide Actuator, Through Hole, Slide Switch"
-			(at 210.82 26.67 0)
-			(effects
-				(font
-					(size 1.27 1.27)
-				)
-				(hide yes)
-			)
-		)
-		(property "Height" "14.5"
-			(at 184.15 421.59 0)
+		(property "Reference" "R34"
+			(at 87.0153 71.2429 90)
 			(effects
 				(font
 					(size 1.27 1.27)
 				)
-				(justify left top)
-				(hide yes)
+				(justify right)
 			)
 		)
-		(property "Mouser Part Number" "179-SLW16781056AND"
-			(at 184.15 521.59 0)
+		(property "Value" "10k"
+			(at 87.0153 68.7029 90)
 			(effects
 				(font
 					(size 1.27 1.27)
 				)
-				(justify left top)
-				(hide yes)
+				(justify right)
 			)
 		)
-		(property "Mouser Price/Stock" "https://www.mouser.co.uk/ProductDetail/Same-Sky/SLW-1678105-6A-N-D?qs=IKkN%2F947nfCWfuHPg7jcWw%3D%3D"
-			(at 184.15 621.59 0)
+		(property "Footprint" "Resistor_SMD:R_1206_3216Metric_Pad1.30x1.75mm_HandSolder"
+			(at 88.9 67.818 90)
 			(effects
 				(font
 					(size 1.27 1.27)
 				)
-				(justify left top)
 				(hide yes)
 			)
 		)
-		(property "Manufacturer_Name" "Same Sky"
-			(at 184.15 721.59 0)
+		(property "Datasheet" "~"
+			(at 88.9 66.04 0)
 			(effects
 				(font
 					(size 1.27 1.27)
 				)
-				(justify left top)
 				(hide yes)
 			)
 		)
-		(property "Manufacturer_Part_Number" "SLW-1678105-6A-N-D"
-			(at 184.15 821.59 0)
+		(property "Description" "Resistor"
+			(at 88.9 66.04 0)
 			(effects
 				(font
 					(size 1.27 1.27)
 				)
-				(justify left top)
 				(hide yes)
 			)
 		)
-		(pin "6"
-		)
-		(pin "3"
-		)
 		(pin "1"
 		)
 		(pin "2"
 		)
-		(pin "5"
-		)
-		(pin "4"
-		)
 		(instances
-			(project ""
+			(project "lighthouse"
 				(path "/7210d03b-7565-45ff-aaca-ad566f37cd67"
-					(reference "S1")
+					(reference "R34")
 					(unit 1)
 				)
@@
 			)
 		)
-		(property "Footprint" "LED_SMD:LED_1206_3216Metric_Pad1.42x1.75mm_HandSolder"
+		(property "Footprint" "LED_THT:LED_D3.0mm"
 			(at 52.07 168.91 0)
 			(effects

Commit message: Finalized the board (experiment pending)
Parts:
- F1, F2: footprint Fuse:Fuse_1206_3216Metric_Pad1.42x1.75mm_HandSolder -> Fuse:Fuse_2920_7451Metric_Pad2.10x5.45mm_HandSolder
Changed lines of the file:
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@@
 			)
 		)
-		(property "Footprint" "Fuse:Fuse_1206_3216Metric_Pad1.42x1.75mm_HandSolder"
+		(property "Footprint" "Fuse:Fuse_2920_7451Metric_Pad2.10x5.45mm_HandSolder"
 			(at 219.71 38.608 90)
 			(effects
@@
 			)
 		)
-		(property "Footprint" "Fuse:Fuse_1206_3216Metric_Pad1.42x1.75mm_HandSolder"
+		(property "Footprint" "Fuse:Fuse_2920_7451Metric_Pad2.10x5.45mm_HandSolder"
 			(at 219.71 28.448 90)
 			(effects
