File: circuits/lighthouse/lighthouse.kicad_pcb (KiCad board)
At the start: 2 copper layers, 83 x 80 mm, 97 parts, among them IC1 SX1308, J1 USB_C_Receptacle_USB2.0_14P, J2 Conn_01x03_Socket, Q1 BC337, Q2 FS8205A, Q3 2N7002K, Q4 BC817-40, Q5 BC817-40, SW1 SW_Push_DPDT, U1 R300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

Commit message: Production ready board
Parts:
- removed D9: D, LED_SMD:LED_1206_3216Metric_Pad1.42x1.75mm_HandSolder
- removed R28, R29: 1k, Resistor_SMD:R_1206_3216Metric_Pad1.30x1.75mm_HandSolder
- removed R30: 10k, Resistor_SMD:R_1206_3216Metric_Pad1.30x1.75mm_HandSolder
- removed SW1: SW_Push_DPDT, Connector_JST:JST_XH_B4B-XH-A_1x04_P2.50mm_Vertical
- removed U10: CP2102-GMR, CP2102-GMR:QFN28_5X5_SIL
- removed U6: AMS1117-3.3, Package_TO_SOT_SMD:SOT-223-3_TabPin2
- added C18: 100n, Capacitor_SMD:C_1206_3216Metric_Pad1.33x1.80mm_HandSolder, F.Cu at (41.0, 90.5)
- added H1: MountingHole_Pad, MountingHole:MountingHole_3.2mm_M3_Pad_Via, F.Cu at (45.1, 122.8)
- added H2: MountingHole_Pad, MountingHole:MountingHole_3.2mm_M3_Pad_Via, F.Cu at (100.8, 122.8)
- added H3: MountingHole, MountingHole:MountingHole_3.2mm_M3, F.Cu at (35.2, 57.5)
- added H4: MountingHole, MountingHole:MountingHole_3.2mm_M3, F.Cu at (77.0, 57.5)
- added IO13: GPIO13, TestPoint:TestPoint_Pad_D1.0mm, F.Cu at (56.5, 83.8)
- added IO14: GPIO14, TestPoint:TestPoint_Pad_D1.0mm, F.Cu at (53.5, 83.8)
- added IO25: GPIO25, TestPoint:TestPoint_Pad_D1.0mm, F.Cu at (44.5, 69.5)
- added IO26: GPIO26, TestPoint:TestPoint_Pad_D1.0mm, F.Cu at (50.5, 83.8)
- added J3: USB_C_Receptacle_PowerOnly_6P, Connector_USB:USB_C_Receptacle_HRO_TYPE-C-31-M-17, F.Cu at (34.1, 87.3)
- added JP1: SolderJumper_2_Bridged, Jumper:SolderJumper-2_P1.3mm_Bridged2Bar_RoundedPad1.0x1.5mm, B.Cu at (89.8, 108.5)
- added JP2: SolderJumper_2_Bridged, Jumper:SolderJumper-2_P1.3mm_Bridged2Bar_RoundedPad1.0x1.5mm, B.Cu at (52.3, 63.4)
- added JP3: SolderJumper_2_Bridged, Jumper:SolderJumper-2_P1.3mm_Bridged2Bar_RoundedPad1.0x1.5mm, B.Cu at (96.3, 93.2)
- added JP4: SolderJumper_2_Open, Jumper:SolderJumper-2_P1.3mm_Open_RoundedPad1.0x1.5mm, B.Cu at (96.3, 95.8)
- added SW2: SW_DPDT_x2, Connector_JST:JST_XH_B4B-XH-A_1x04_P2.50mm_Vertical, F.Cu at (43.4, 97.5)
- added TP1: TestPoint, TestPoint:TestPoint_Pad_D1.0mm, F.Cu at (47.5, 93.0)
- added TP2: TestPoint, TestPoint:TestPoint_Pad_D1.0mm, F.Cu at (105.8, 109.8)
- added TP3: TestPoint, TestPoint:TestPoint_Pad_D1.0mm, F.Cu at (72.8, 93.2)
- added TP4: TestPoint, TestPoint:TestPoint_Pad_D1.0mm, F.Cu at (38.5, 61.8)
- added TP5: RX, TestPoint:TestPoint_Pad_D1.0mm, F.Cu at (83.0, 83.2)
- added TP6: TX, TestPoint:TestPoint_Pad_D1.0mm, F.Cu at (81.2, 81.2)
- added TP7: TestPoint, TestPoint:TestPoint_Pad_D1.0mm, F.Cu at (113.2, 89.8)
- added TP8: TestPoint, TestPoint:TestPoint_Pad_D1.0mm, F.Cu at (105.8, 100.2)
- BZ1: footprint Buzzer_Beeper:MagneticBuzzer_PUI_AT-0927-TT-6-R -> Buzzer_Beeper:Buzzer_12x9.5RM7.6
- C10: value 56n -> 22uF
- C4: value 10u -> 22u
- D10: value D -> SS24A; footprint LED_SMD:LED_1206_3216Metric_Pad1.42x1.75mm_HandSolder -> Diode_SMD:D_SMA
- D12, D7: value D_Schottky -> SS24A; footprint Diode_SMD:D_2114_3652Metric_Pad1.85x3.75mm_HandSolder -> Diode_SMD:D_SMA
- D5, D6: value D -> LED
- J1: value USB_C_Receptacle_USB2.0_14P -> Conn_01x06_Socket; footprint Connector_USB:USB_C_Receptacle_G-Switch_GT-USB-7010ASV -> Connector_PinHeader_2.00mm:PinHeader_2x03_P2.00mm_Vertical
- L1: footprint Inductor_THT:L_Radial_L8.0mm_W8.0mm_P5.00mm_Neosid_SD8 -> IDCP2218ER101M01:IDCP2218ER101M01
- R14: value 220 -> 1k
- R3: value 820 -> 1k
- R37, R9: value 47k -> 120k
- R5: value 100 (470) -> 150
- U2: value AMS1117-3.3 -> TS1117B
- moved J1 28.9 mm to (63.5, 83.9)
- moved D6 24.5 mm to (49.0, 109.7), turned to 0 degrees
- moved R1 19.0 mm to (49.0, 107.0), turned to 0 degrees
- moved C7 14.9 mm to (102.0, 97.2)
- moved D10 14.4 mm to (102.2, 107.2), turned to 90 degrees
- moved R17 12.2 mm to (92.0, 90.2), turned to 0 degrees
- moved D11 9.06 mm to (110.3, 109.5)
- moved C10 8.57 mm to (40.9, 84.2)
- moved D15 7.88 mm to (54.0, 87.0)
- moved R3 7.31 mm to (49.2, 95.6), turned to 180 degrees
- moved F1 7.00 mm to (36.2, 106.0)
- moved F2 7.00 mm to (43.0, 106.0)
- moved Q3 6.69 mm to (101.6, 101.5)
- moved R2 6.33 mm to (54.2, 107.0), turned to 180 degrees
- moved C9 5.86 mm to (110.2, 101.4), turned to 180 degrees
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Connections:
- BZ1 pad 1: +5V -> /R300/5V
- C10 pad 1: GND -> Net-(C10-Pad1)
- C10 pad 2: Net-(U10-VDD) -> GND
- C15 pad 1: +5V -> /R300/5V
- C16 pad 1: +3.3V -> Net-(JP2-B)
- C6 pad 2: +5V -> /R300/5V
- C7 pad 2: +5V -> /R300/5V
- C8 pad 1: +5V -> /R300/5V
- C9 pad 1: +5V -> /R300/5V
- D10 pad 1: +5V -> /R300/5V
- D11 pad 2: +5V -> /R300/5V
- D16 pad 2: Net-(D16-A) -> /Charger/VIN
- F1 pad 1: Net-(F1-Pad1) -> Net-(C10-Pad1)
- F1 pad 2: Net-(D16-A) -> Net-(SW2A-B)
- F2 pad 1: Net-(SW1-A) -> /Charger/+BAT
- F2 pad 2: Net-(D15-A) -> Net-(SW2B-B)
- Q1 pad 3: /R300/GND -> Net-(JP3-A)
- R15 pad 1: +5V -> /R300/5V
- R32 pad 1: /Charger/CC2 -> Net-(J3-CC2)
- R33 pad 1: /Charger/CC1 -> Net-(J3-CC1)
- U1 pad 12: Net-(D9-A) -> TX
- U1 pad 9: +5V -> /R300/5V
- U7 pad 13: unconnected-(U7-IO14-Pad13) -> Net-(U7-IO14)
- U7 pad 2: +3.3V -> Net-(JP2-B)
Routing:
- net GND: track 134.6 -> 27.6 mm, vias 19 -> 29
- net /R300/5V: track 0.00 -> 80.1 mm, vias 0 -> 2
- net +5V: track 133.9 -> 71.1 mm
- net Net-(C10-Pad1): track 0.00 -> 43.6 mm, vias 0 -> 1
- net /Charger/VIN: track 93.4 -> 60.5 mm
- net Net-(JP2-B): track 0.00 -> 22.2 mm
- net Net-(Q3-G): track 6.36 -> 28.5 mm, vias 0 -> 2
- net Net-(U10-D-): track 19.8 -> 0.00 mm
- net Net-(U10-D+): track 18.7 -> 0.00 mm, vias 2 -> 0
- net Net-(D16-A): track 18.0 -> 0.00 mm
- net MP28: track 15.6 -> 32.8 mm, vias 2 -> 1
- net +3.3V: track 174.5 -> 157.4 mm, vias 8 -> 6
- net unconnected-(IO25-Pad1): track 0.00 -> 16.2 mm, vias 0 -> 2
- net Net-(U10-TXD): track 15.5 -> 0.00 mm, vias 2 -> 0
- net Net-(U4-~{STDBY}): track 19.3 -> 4.18 mm, vias 2 -> 0
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- added copper zone on F.Cu, net GND
Other:
- board text added: "3v3"
- board text added: "5V"
- board text added: "GND"
- board text added: "I5V"
- board text added: "IGND"
- board text added: "VIN"

Commit message: Patched board issue, next board order will need it applied
Connections:
- JP3 pad 1: Net-(JP3-A) -> RFID_PW_SENSE
- Q1 pad 3: Net-(JP3-A) -> RFID_PW_SENSE
Routing:
- net Net-(JP3-A): track 3.46 -> 0.00 mm
- net RFID_PW_SENSE: track 32.5 -> 36.0 mm
Changed lines of the file:
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@@
 	(net 87 "/R300/5V")
 	(net 88 "Net-(JP2-B)")
-	(net 89 "Net-(JP3-A)")
 	(footprint "Resistor_SMD:R_1206_3216Metric_Pad1.30x1.75mm_HandSolder"
 		(layer "F.Cu")
@@
 		(model "${KIPRJMOD}/components/36911000000--3DModel-STEP-510211.STEP"
 			(offset
-				(xyz 0 0 0)
+				(xyz 0 0 -0.5)
 			)
 			(scale
@@
 		(attr smd)
 		(fp_line
+			(start -2.286 -1.016)
+			(end 2.286 1.016)
+			(stroke
+				(width 0.1)
+				(type default)
+			)
+			(layer "F.SilkS")
+		)
+		(fp_line
 			(start -0.727064 -0.91)
 			(end 0.727064 -0.91)
@@
 			(layer "F.SilkS")
 		)
+		(fp_line
+			(start 2.286 -1.016)
+			(end -2.286 1.016)
+			(stroke
+				(width 0.1)
+				(type default)
+			)
+			(layer "F.SilkS")
+		)
 		(fp_rect
 			(start -2.45 -1.13)
@@
 		)
 		(embedded_fonts no)
-		(model "${KICAD9_3DMODEL_DIR}/Resistor_SMD.3dshapes/R_1206_3216Metric.step"
-			(offset
-				(xyz 0 0 0)
-			)
-			(scale
-				(xyz 1 1 1)
-			)
-			(rotate
-				(xyz 0 0 0)
-			)
-		)
 	)
 	(footprint "Capacitor_SMD:C_1206_3216Metric_Pad1.33x1.80mm_HandSolder"
@@
 		(model "${KICAD9_3DMODEL_DIR}/LED_THT.3dshapes/LED_D3.0mm.step"
 			(offset
-				(xyz 0 0 0)
+				(xyz 0 0 -3)
 			)
 			(scale
@@
 			)
 			(rotate
-				(xyz 0 0 0)
+				(xyz -0 -0 -0)
 			)
 		)
@@
 		(model "${KICAD9_3DMODEL_DIR}/LED_THT.3dshapes/LED_D3.0mm.step"
 			(offset
-				(xyz 0 0 0)
+				(xyz 0 0 -3)
 			)
 			(scale
@@
 			)
 			(rotate
-				(xyz 0 0 0)
+				(xyz -0 -0 -0)
 			)
 		)
@@
 		(model "${KICAD9_3DMODEL_DIR}/Battery.3dshapes/BatteryHolder_MPD_BH-18650-PC2.step"
 			(offset
-				(xyz 0 0 0)
+				(xyz 0 0 -0.2)
 			)
 			(scale
@@
 			)
 			(rotate
-				(xyz 0 0 0)
+				(xyz -0 -0 -0)
 			)
 		)
@@
 		(attr smd)
 		(fp_line
+			(start 2.286 -1.016)
+			(end -2.286 1.016)
+			(stroke
+				(width 0.1)
+				(type default)
+			)
+			(layer "F.SilkS")
+		)
+		(fp_line
 			(start -0.727064 0.91)
 			(end 0.727064 0.91)
@@
 			(layer "F.SilkS")
 		)
+		(fp_line
+			(start -2.286 -1.016)
+			(end 2.286 1.016)
+			(stroke
+				(width 0.1)
+				(type default)
+			)
+			(layer "F.SilkS")
+		)
 		(fp_rect
 			(start -2.45 -1.13)
@@
 		)
 		(embedded_fonts no)
-		(model "${KICAD9_3DMODEL_DIR}/Resistor_SMD.3dshapes/R_1206_3216Metric.step"
-			(offset
-				(xyz 0 0 0)
-			)
-			(scale
-				(xyz 1 1 1)
-			)
-			(rotate
-				(xyz 0 0 0)
-			)
-		)
 	)
 	(footprint "MountingHole:MountingHole_3.2mm_M3"
@@
 		(model "/media/kuba/Games/Documents/VUT/bachelor/circuits/lighthouse/components/YR300/YR300.step"
 			(offset
-				(xyz 0 -13 0)
+				(xyz 0 -13 -1.7)
 			)
 			(scale
@@
 		(model "${KIPRJMOD}/components/36911000000--3DModel-STEP-510211.STEP"
 			(offset
-				(xyz 0 0 0)
+				(xyz 0 0 -0.5)
 			)
 			(scale
@@
 		(model "${KICAD9_3DMODEL_DIR}/LED_THT.3dshapes/LED_D3.0mm.step"
 			(offset
-				(xyz 0 0 0)
+				(xyz 0 0 -3)
 			)
 			(scale
@@
 			)
 			(rotate
-				(xyz 0 0 0)
+				(xyz -0 -0 -0)
 			)
 		)
@@
 		(model "/media/kuba/Games/Documents/VUT/bachelor/circuits/lighthouse/components/LIB_3296W-1-103LF/3296W-1-103LF.stp"
 			(offset
-				(xyz 2.25 2 11)
+				(xyz 2.25 2 10)
 			)
 			(scale
@@
 			(layers "*.Cu" "*.Mask")
 			(remove_unused_layers no)
-			(net 89 "Net-(JP3-A)")
+			(net 68 "RFID_PW_SENSE")
 			(pinfunction "C")
 			(pintype "passive")
@@
 		(model "${KICAD9_3DMODEL_DIR}/LED_THT.3dshapes/LED_D3.0mm.step"
 			(offset
-				(xyz 0 0 0)
+				(xyz 0 0 -3)
 			)
 			(scale
@@
 			)
 			(rotate
-				(xyz 0 0 0)
+				(xyz -0 -0 -0)
 			)
 		)
@@
 		(tags "net tie solder jumper bridged")
 		(property "Reference" "JP3"
-			(at 0 1.8 0)
+			(at 0 -1.7 0)
 			(layer "B.SilkS")
 			(effects
@@
 			(size 1 0.5)
 			(layers "B.Cu" "B.Mask")
-			(net 89 "Net-(JP3-A)")
+			(net 68 "RFID_PW_SENSE")
 			(pinfunction "A")
 			(pintype "passive")
@@
 	)
 	(segment
+		(start 92.28 93.2)
+		(end 92.25 93.23)
+		(width 0.2)
+		(layer "B.Cu")
+		(net 68)
+	)
+	(segment
 		(start 78.25 81)
 		(end 85 87.75)
@@
 	)
 	(segment
+		(start 95.7 93.2)
+		(end 92.28 93.2)
+		(width 1)
+		(layer "B.Cu")
+		(net 68)
+	)
+	(segment
 		(start 75.04 81)
 		(end 78.25 81)
@@
 		(net 88)
 	)
-	(segment
-		(start 92.28 93.2)
-		(end 92.25 93.23)
-		(width 0.2)
-		(layer "B.Cu")
-		(net 89)
-	)
-	(segment
-		(start 95.7 93.2)
-		(end 92.28 93.2)
-		(width 1)
-		(layer "B.Cu")
-		(net 89)
-	)
 	(zone
