File: circuits/lighthouse/charger.kicad_sch (KiCad schematic)
At the start: 13 parts, among them Q2 FS8205A, U4 TP4056-42-ESOP8, U5 DW01A

Commit message: Schematic title block
Other:
- company: (none) -> Brno University of Technology
- title: (none) -> Charger submodule
Changed lines of the file:
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@@
 	(generator_version "9.0")
 	(paper "A5")
+	(title_block
+		(title "Charger submodule")
+		(date "2026-03-25")
+		(rev "1")
+		(company "Brno University of Technology")
+		(comment 1 "Embedded Implementation of an Attendance System for Integration")
+		(comment 2 "into an Enterprise Application")
+		(comment 3 "Author: Jakub Hloušek")
+		(comment 4 "Supervisor: Ing. Michal Bastl, Ph.D")
+	)
 	(junction
 		(at 166.37 36.83)
